File: T512CLK.kicad_pcb (KiCad board)
At the start: 2 copper layers, 145.1 x 107.5 mm, 60 parts, among them J1 Bus_ISA_8bit, U1 41256, U10 41256, U11 41256, U12 41256, U13 41256, U14 41256, U15 41256, U16 41256, U17 74LS139, U18 74LS08, U19 74LS32, U2 41256, U20 74LS258, U21 74LS258, U22 RTC, U23 74LS138, U24 74LS373, U25 8237A, U26 74LS245, U27 74LS74, U28 74LS04, U29 74LS245, U3 41256, U30 74LS670, U31 74LS00, U32 74LS74, U4 41256, U5 41256, U6 41256, U7 41256, U8 41256, U9 41256

Commit message: Change RP3 symbol from a single to split for better readability.
Connections:
- net /~MEMR~_DRV renamed /~MEMR~_BUF
- net /~MEMW~_DRV renamed /~MEMW~_BUF
- net A0_DRV renamed A0_BUF
- net A1_DRV renamed A1_BUF
- net A2_DRV renamed A2_BUF
- net A3_DRV renamed A3_BUF
- net IO_OR_MEM_READ renamed /IO_OR_MEM_READ
- net ~EOP renamed /~EOP
- net ~IOR~_DRV renamed ~IOR~_BUF
- net ~IOW~_DRV renamed ~IOW~_BUF
- RP3 pad 8: Net-(RP3-Pad8) -> (no net)
